File: E1S.kicad_pcb (KiCad board)
At the start: 2 copper layers, 61.2 x 34.5 mm, 3 parts

Commit message: shrinking
Parts:
- moved C1 6.61 mm to (165.6, 90.4)
Connections:
- C2 pad 1: R_AUD -> A_GND
- C2 pad 3: A_GND -> R_AUD
Routing:
- net BLUE: track 32.3 -> 0.00 mm
- net A_GND: track 28.6 -> 0.00 mm
- net GREEN: track 27.1 -> 0.00 mm
- net SYNC: track 22.2 -> 0.00 mm
- net R_AUD: track 23.3 -> 1.10 mm
- net L_AUD: track 19.4 -> 0.00 mm
- net RED: track 16.1 -> 0.00 mm
- removed copper zone on B.Cu, net GND
- removed copper zone on F.Cu, net GND
Other:
- board outline removed
